Commit message: fix xacro warnings

File: urdf/base_hub.urdf.xacro (robot description, xacro)
@@ -2,7 +2,7 @@
 <robot name="base_hub" xmlns:xacro="http://www.ros.org/wiki/xacro">
     <!-- Macro for calculating inertia of cylinder -->
-    <macro name="cylinder_inertia" params="m r h">
+    <xacro:macro name="cylinder_inertia" params="m r h">
         <inertia ixx="${m*(3*r*r+h*h)/12}" ixy="0" ixz="0" iyy="${m*(3*r*r+h*h)/12}" iyz="0" izz="${m*r*r/2}"/>
-    </macro>
+    </xacro:macro>
     <xacro:macro name="base_hub" params="multi_hub hub_id parent x y z roll pitch yaw">
       <xacro:if value="${multi_hub}">
@@ -26,5 +26,5 @@
                   <mass value="0.013"/>
                   <origin xyz="0 0 0"/>
-                  <cylinder_inertia m="0.013" r="0.06" h="0.03" />
+                  <xacro:cylinder_inertia m="0.013" r="0.06" h="0.03" />
               </inertial>
           </link>
@@ -64,5 +64,5 @@
                   <mass value="0.013"/>
                   <origin xyz="0 0 0"/>
-                  <cylinder_inertia m="0.013" r="0.06" h="0.03" />
+                  <xacro:cylinder_inertia m="0.013" r="0.06" h="0.03" />
               </inertial>
           </link>

File: urdf/teraranger_evo_tower.urdf.xacro (robot description, xacro)
@@ -5,14 +5,14 @@
     <xacro:macro name="teraranger_evo_tower" params="multi_hub hub_id parent x y z roll pitch yaw">
       <!-- EVO TOWER CONFIG-->
-      <base_hub multi_hub="${multi_hub}" hub_id='${hub_id}' parent="${parent}" x="${x}" y="${y}" z="${z}" roll="${roll}" pitch="${pitch}" yaw="${yaw}" />
+      <xacro:base_hub multi_hub="${multi_hub}" hub_id='${hub_id}' parent="${parent}" x="${x}" y="${y}" z="${z}" roll="${roll}" pitch="${pitch}" yaw="${yaw}" />
       <!--<base_hub multi_hub="0" hub_id='0' parent="base_link" x="0" y="0" z="0.26" roll="0" pitch="0" yaw="0"/>-->
-      <teraranger_evo multi_hub="0" hub_id='0' id="0" x="0.046" y="0.000" z="0" roll="0" pitch="0" yaw="0.000" gaussian_noise="0"/>
-      <teraranger_evo multi_hub="0" hub_id='0' id="1" x="0.032" y="-0.032" z="0" roll="0" pitch="0" yaw="-0.785" gaussian_noise="0"/>
-      <teraranger_evo multi_hub="0" hub_id='0' id="2" x="0.000" y="-0.046" z="0" roll="0" pitch="0" yaw="-1.571" gaussian_noise="0"/>
-      <teraranger_evo multi_hub="0" hub_id='0' id="3" x="-0.032" y="-0.032" z="0" roll="0" pitch="0" yaw="-2.356" gaussian_noise="0"/>
-      <teraranger_evo multi_hub="0" hub_id='0' id="4" x="-0.046" y="0.000" z="0" roll="0" pitch="0" yaw="3.142" gaussian_noise="0"/>
-      <teraranger_evo multi_hub="0" hub_id='0' id="5" x="-0.032" y="0.032" z="0" roll="0" pitch="0" yaw="2.356" gaussian_noise="0"/>
-      <teraranger_evo multi_hub="0" hub_id='0' id="6" x="0.000" y="0.046" z="0" roll="0" pitch="0" yaw="1.571" gaussian_noise="0"/>
-      <teraranger_evo multi_hub="0" hub_id='0' id="7" x="0.032" y="0.032" z="0" roll="0" pitch="0" yaw="0.785" gaussian_noise="0"/>
+      <xacro:teraranger_evo multi_hub="0" hub_id='0' id="0" x="0.046" y="0.000" z="0" roll="0" pitch="0" yaw="0.000" gaussian_noise="0"/>
+      <xacro:teraranger_evo multi_hub="0" hub_id='0' id="1" x="0.032" y="-0.032" z="0" roll="0" pitch="0" yaw="-0.785" gaussian_noise="0"/>
+      <xacro:teraranger_evo multi_hub="0" hub_id='0' id="2" x="0.000" y="-0.046" z="0" roll="0" pitch="0" yaw="-1.571" gaussian_noise="0"/>
+      <xacro:teraranger_evo multi_hub="0" hub_id='0' id="3" x="-0.032" y="-0.032" z="0" roll="0" pitch="0" yaw="-2.356" gaussian_noise="0"/>
+      <xacro:teraranger_evo multi_hub="0" hub_id='0' id="4" x="-0.046" y="0.000" z="0" roll="0" pitch="0" yaw="3.142" gaussian_noise="0"/>
+      <xacro:teraranger_evo multi_hub="0" hub_id='0' id="5" x="-0.032" y="0.032" z="0" roll="0" pitch="0" yaw="2.356" gaussian_noise="0"/>
+      <xacro:teraranger_evo multi_hub="0" hub_id='0' id="6" x="0.000" y="0.046" z="0" roll="0" pitch="0" yaw="1.571" gaussian_noise="0"/>
+      <xacro:teraranger_evo multi_hub="0" hub_id='0' id="7" x="0.032" y="0.032" z="0" roll="0" pitch="0" yaw="0.785" gaussian_noise="0"/>
    </xacro:macro>
 </robot>

File: urdf/teraranger_tower.urdf.xacro (robot description, xacro)
@@ -4,13 +4,13 @@
     <xacro:include filename="$(find teraranger_description)/urdf/teraranger_one.urdf.xacro"/>
     <xacro:macro name="teraranger_tower" params="multi_hub hub_id parent x y z roll pitch yaw">
-        <base_hub multi_hub="${multi_hub}" hub_id='${hub_id}' parent="${parent}" x="${x}" y="${y}" z="${z}" roll="${roll}" pitch="${pitch}" yaw="${yaw}" />
-        <teraranger_one multi_hub="${multi_hub}" hub_id='${hub_id}' id="0" x="0.060" y="0.000" z="0.0" roll="0.0" pitch="0.0" yaw="0.000" gaussian_noise="0.06"/>
-        <teraranger_one multi_hub="${multi_hub}" hub_id='${hub_id}' id="1" x="0.042" y="0.042" z="0.0" roll="0.0" pitch="0.0" yaw="0.785" gaussian_noise="0.06"/>
-        <teraranger_one multi_hub="${multi_hub}" hub_id='${hub_id}' id="2" x="0.000" y="0.060" z="0.0" roll="0.0" pitch="0.0" yaw="1.571" gaussian_noise="0.06"/>
-        <teraranger_one multi_hub="${multi_hub}" hub_id='${hub_id}' id="3" x="-0.042" y="0.042" z="0.0" roll="0.0" pitch="0.0" yaw="2.356" gaussian_noise="0.06"/>
-        <teraranger_one multi_hub="${multi_hub}" hub_id='${hub_id}' id="4" x="-0.060" y="0.000" z="0.0" roll="0.0" pitch="0.0" yaw="3.14" gaussian_noise="0.06"/>
-        <teraranger_one multi_hub="${multi_hub}" hub_id='${hub_id}' id="5" x="-0.042" y="-0.042" z="0.0" roll="0.0" pitch="0.0" yaw="-2.356" gaussian_noise="0.06"/>
-        <teraranger_one multi_hub="${multi_hub}" hub_id='${hub_id}' id="6" x="0.000" y="-0.060" z="0.0" roll="0.0" pitch="0.0" yaw="-1.571" gaussian_noise="0.06"/>
-        <teraranger_one multi_hub="${multi_hub}" hub_id='${hub_id}' id="7" x="0.042" y="-0.042" z="0.0" roll="0.0" pitch="0.0" yaw="-0.785" gaussian_noise="0.06"/>
+        <xacro:base_hub multi_hub="${multi_hub}" hub_id='${hub_id}' parent="${parent}" x="${x}" y="${y}" z="${z}" roll="${roll}" pitch="${pitch}" yaw="${yaw}" />
+        <xacro:teraranger_one multi_hub="${multi_hub}" hub_id='${hub_id}' id="0" x="0.060" y="0.000" z="0.0" roll="0.0" pitch="0.0" yaw="0.000" gaussian_noise="0.06"/>
+        <xacro:teraranger_one multi_hub="${multi_hub}" hub_id='${hub_id}' id="1" x="0.042" y="0.042" z="0.0" roll="0.0" pitch="0.0" yaw="0.785" gaussian_noise="0.06"/>
+        <xacro:teraranger_one multi_hub="${multi_hub}" hub_id='${hub_id}' id="2" x="0.000" y="0.060" z="0.0" roll="0.0" pitch="0.0" yaw="1.571" gaussian_noise="0.06"/>
+        <xacro:teraranger_one multi_hub="${multi_hub}" hub_id='${hub_id}' id="3" x="-0.042" y="0.042" z="0.0" roll="0.0" pitch="0.0" yaw="2.356" gaussian_noise="0.06"/>
+        <xacro:teraranger_one multi_hub="${multi_hub}" hub_id='${hub_id}' id="4" x="-0.060" y="0.000" z="0.0" roll="0.0" pitch="0.0" yaw="3.14" gaussian_noise="0.06"/>
+        <xacro:teraranger_one multi_hub="${multi_hub}" hub_id='${hub_id}' id="5" x="-0.042" y="-0.042" z="0.0" roll="0.0" pitch="0.0" yaw="-2.356" gaussian_noise="0.06"/>
+        <xacro:teraranger_one multi_hub="${multi_hub}" hub_id='${hub_id}' id="6" x="0.000" y="-0.060" z="0.0" roll="0.0" pitch="0.0" yaw="-1.571" gaussian_noise="0.06"/>
+        <xacro:teraranger_one multi_hub="${multi_hub}" hub_id='${hub_id}' id="7" x="0.042" y="-0.042" z="0.0" roll="0.0" pitch="0.0" yaw="-0.785" gaussian_noise="0.06"/>
     </xacro:macro>
 </robot>
