Commit message: fix bug frame naming

File: urdf/teraranger_evo.urdf.xacro (robot description, xacro)
@@ -26,5 +26,5 @@
               </inertial>
             </link>
-            <joint name="inertial_joint_${hub_id}" type="fixed">
+            <joint name="inertial_joint_${hub_id}_base_range_joint_${id}" type="fixed">
               <origin xyz="0.0 0.0 0" rpy="0 0 0" />
               <parent link="base_hub_${hub_id}"/>
@@ -90,5 +90,5 @@
               </inertial>
             </link>
-            <joint name="inertial_joint_${hub_id}" type="fixed">
+            <joint name="inertial_joint_base_range_joint_${id}" type="fixed">
               <origin xyz="0.0 0.0 0" rpy="0 0 0" />
               <parent link="base_hub"/>

File: urdf/teraranger_one.urdf.xacro (robot description, xacro)
@@ -24,5 +24,5 @@
               </inertial>
             </link>
-            <joint name="inertial_joint_${hub_id}" type="fixed">
+            <joint name="inertial_joint_${hub_id}_base_range_joint_${id}" type="fixed">
               <origin xyz="0.0 0.0 0" rpy="0 0 0" />
               <parent link="base_hub_${hub_id}"/>
@@ -88,5 +88,5 @@
               </inertial>
             </link>
-            <joint name="inertial_joint_${hub_id}" type="fixed">
+            <joint name="inertial_joint_base_range_joint_${id}" type="fixed">
               <origin xyz="0.0 0.0 0" rpy="0 0 0" />
               <parent link="base_hub"/>

Commit message: fix single sensor launch + refactor names

File: urdf/teraranger_evo.urdf.xacro (robot description, xacro)
@@ -1,6 +1,7 @@
 <?xml version="1.0"?>
 <robot name="teraranger_evo" xmlns:xacro="http://www.ros.org/wiki/xacro">
-    <xacro:macro name="teraranger_evo" params="multi_hub hub_id id x y z roll pitch yaw gaussian_noise">
+    <xacro:macro name="teraranger_evo" params="multi_hub hub_id id x y z roll pitch yaw gaussian_noise parent:=base_hub_">
         <xacro:if value="${multi_hub}">
+            <xacro:property name="hub_parent" value="${parent}${hub_id}"/>
             <link name="hub_${hub_id}_base_range_${id}">
                 <visual>
@@ -16,5 +17,5 @@
             <joint name="hub_${hub_id}_base_range_joint_${id}" type="fixed">
                 <origin xyz="${x} ${y} ${z}" rpy="${roll} ${pitch} ${yaw}"/>
-                <parent link="base_hub_${hub_id}"/>
+                <parent link="${hub_parent}"/>
                 <child link="hub_${hub_id}_base_range_${id}"/>
             </joint>
@@ -28,5 +29,5 @@
             <joint name="inertial_joint_${hub_id}_base_range_joint_${id}" type="fixed">
               <origin xyz="0.0 0.0 0" rpy="0 0 0" />
-              <parent link="base_hub_${hub_id}"/>
+              <parent link="${hub_parent}"/>
               <child link="inertial_link_${hub_id}_base_range_joint_${id}"/>
             </joint>
@@ -75,10 +76,12 @@
                         <mesh filename="package://teraranger_description/meshes/teraranger_evo.stl"/>
                     </geometry>
-                    <material name="Yellow"/>
+                    <material name="Yellow">
+                        <color rgba="1.0 1.0 0.0 1.0"/>
+                    </material>
                 </visual>
             </link>
             <joint name="base_range_joint_${id}" type="fixed">
                 <origin xyz="${x} ${y} ${z}" rpy="${roll} ${pitch} ${yaw}"/>
-                <parent link="base_hub"/>
+                <parent link="${parent}"/>
                 <child link="base_range_${id}"/>
             </joint>
@@ -92,5 +95,5 @@
             <joint name="inertial_joint_base_range_joint_${id}" type="fixed">
               <origin xyz="0.0 0.0 0" rpy="0 0 0" />
-              <parent link="base_hub"/>
+              <parent link="${parent}"/>
               <child link="inertial_link_base_range_joint_${id}"/>
             </joint>

File: urdf/teraranger_evo_tower.urdf.xacro (robot description, xacro)
@@ -5,14 +5,13 @@
     <xacro:macro name="teraranger_evo_tower" params="multi_hub hub_id parent x y z roll pitch yaw">
       <!-- EVO TOWER CONFIG-->
-      <xacro:base_hub multi_hub="${multi_hub}" hub_id='${hub_id}' parent="${parent}" x="${x}" y="${y}" z="${z}" roll="${roll}" pitch="${pitch}" yaw="${yaw}" />
-      <!--<base_hub multi_hub="0" hub_id='0' parent="base_link" x="0" y="0" z="0.26" roll="0" pitch="0" yaw="0"/>-->
-      <xacro:teraranger_evo multi_hub="0" hub_id='0' id="0" x="0.046" y="0.000" z="0" roll="0" pitch="0" yaw="0.000" gaussian_noise="0"/>
-      <xacro:teraranger_evo multi_hub="0" hub_id='0' id="1" x="0.032" y="-0.032" z="0" roll="0" pitch="0" yaw="-0.785" gaussian_noise="0"/>
-      <xacro:teraranger_evo multi_hub="0" hub_id='0' id="2" x="0.000" y="-0.046" z="0" roll="0" pitch="0" yaw="-1.571" gaussian_noise="0"/>
-      <xacro:teraranger_evo multi_hub="0" hub_id='0' id="3" x="-0.032" y="-0.032" z="0" roll="0" pitch="0" yaw="-2.356" gaussian_noise="0"/>
-      <xacro:teraranger_evo multi_hub="0" hub_id='0' id="4" x="-0.046" y="0.000" z="0" roll="0" pitch="0" yaw="3.142" gaussian_noise="0"/>
-      <xacro:teraranger_evo multi_hub="0" hub_id='0' id="5" x="-0.032" y="0.032" z="0" roll="0" pitch="0" yaw="2.356" gaussian_noise="0"/>
-      <xacro:teraranger_evo multi_hub="0" hub_id='0' id="6" x="0.000" y="0.046" z="0" roll="0" pitch="0" yaw="1.571" gaussian_noise="0"/>
-      <xacro:teraranger_evo multi_hub="0" hub_id='0' id="7" x="0.032" y="0.032" z="0" roll="0" pitch="0" yaw="0.785" gaussian_noise="0"/>
+      <xacro:base_hub multi_hub="1" hub_id='${hub_id}' parent="${parent}" x="${x}" y="${y}" z="${z}" roll="${roll}" pitch="${pitch}" yaw="${yaw}" />
+      <xacro:teraranger_evo multi_hub="1" hub_id='0' id="0" x="0.046" y="0.000" z="0" roll="0" pitch="0" yaw="0.000" gaussian_noise="0"/>
+      <xacro:teraranger_evo multi_hub="1" hub_id='0' id="1" x="0.032" y="-0.032" z="0" roll="0" pitch="0" yaw="-0.785" gaussian_noise="0"/>
+      <xacro:teraranger_evo multi_hub="1" hub_id='0' id="2" x="0.000" y="-0.046" z="0" roll="0" pitch="0" yaw="-1.571" gaussian_noise="0"/>
+      <xacro:teraranger_evo multi_hub="1" hub_id='0' id="3" x="-0.032" y="-0.032" z="0" roll="0" pitch="0" yaw="-2.356" gaussian_noise="0"/>
+      <xacro:teraranger_evo multi_hub="1" hub_id='0' id="4" x="-0.046" y="0.000" z="0" roll="0" pitch="0" yaw="3.142" gaussian_noise="0"/>
+      <xacro:teraranger_evo multi_hub="1" hub_id='0' id="5" x="-0.032" y="0.032" z="0" roll="0" pitch="0" yaw="2.356" gaussian_noise="0"/>
+      <xacro:teraranger_evo multi_hub="1" hub_id='0' id="6" x="0.000" y="0.046" z="0" roll="0" pitch="0" yaw="1.571" gaussian_noise="0"/>
+      <xacro:teraranger_evo multi_hub="1" hub_id='0' id="7" x="0.032" y="0.032" z="0" roll="0" pitch="0" yaw="0.785" gaussian_noise="0"/>
    </xacro:macro>
 </robot>

File: urdf/teraranger_one.urdf.xacro (robot description, xacro)
@@ -1,6 +1,7 @@
 <?xml version="1.0"?>
 <robot name="teraranger_one" xmlns:xacro="http://www.ros.org/wiki/xacro">
-    <xacro:macro name="teraranger_one" params="multi_hub hub_id id x y z roll pitch yaw gaussian_noise">
+    <xacro:macro name="teraranger_one" params="multi_hub hub_id id x y z roll pitch yaw gaussian_noise parent:=base_hub_">
         <xacro:if value="${multi_hub}">
+            <xacro:property name="hub_parent" value="${parent}${hub_id}"/>
             <link name="hub_${hub_id}_base_range_${id}">
                 <visual>
@@ -14,5 +15,5 @@
             <joint name="hub_${hub_id}_base_range_joint_${id}" type="fixed">
                 <origin xyz="${x} ${y} ${z}" rpy="${roll} ${pitch} ${yaw}"/>
-                <parent link="base_hub_${hub_id}"/>
+                <parent link="${hub_parent}"/>
                 <child link="hub_${hub_id}_base_range_${id}"/>
             </joint>
@@ -26,5 +27,5 @@
             <joint name="inertial_joint_${hub_id}_base_range_joint_${id}" type="fixed">
               <origin xyz="0.0 0.0 0" rpy="0 0 0" />
-              <parent link="base_hub_${hub_id}"/>
+              <parent link="${hub_parent}"/>
               <child link="inertial_link_${hub_id}_base_range_joint_${id}"/>
             </joint>
@@ -78,5 +79,5 @@
             <joint name="base_range_joint_${id}" type="fixed">
                 <origin xyz="${x} ${y} ${z}" rpy="${roll} ${pitch} ${yaw}"/>
-                <parent link="base_hub"/>
+                <parent link="${parent}"/>
                 <child link="base_range_${id}"/>
             </joint>
@@ -90,5 +91,5 @@
             <joint name="inertial_joint_base_range_joint_${id}" type="fixed">
               <origin xyz="0.0 0.0 0" rpy="0 0 0" />
-              <parent link="base_hub"/>
+              <parent link="${parent}"/>
               <child link="inertial_link_base_range_joint_${id}"/>
             </joint>

Commit message: mods

File: urdf/teraranger_evo.urdf.xacro (robot description, xacro)
@@ -95,5 +95,5 @@
             <joint name="inertial_joint_base_range_joint_${id}" type="fixed">
               <origin xyz="0.0 0.0 0" rpy="0 0 0" />
-              <parent link="${parent}"/>
+              <parent link="base_range_${id}"/>
               <child link="inertial_link_base_range_joint_${id}"/>
             </joint>
